Commit message: a

File: description/robot.urdf.xacro (robot description, xacro)
@@ -1,4 +1,4 @@
 <?xml version="1.0"?>
 <robot xmlns:xacro="http://www.ros.org/wiki/xacro"  name="robot">
-    <xacro:include filenam="robot_core.xacro" />
-</robot>
+    <xacro:include filename ="robot_core.xacro"/>
+</robot>   <link name="base_link"></link>

Commit message: a

File: description/robot.urdf.xacro (robot description, xacro)
@@ -2,3 +2,3 @@
 <robot xmlns:xacro="http://www.ros.org/wiki/xacro"  name="robot">
     <xacro:include filename ="robot_core.xacro"/>
-</robot>   <link name="base_link"></link>
+</robot>
